Commit message: update urdf with collada meshes

File: urdf/jetson.xacro (robot description, xacro)
@@ -26,5 +26,6 @@
       <origin xyz="0 0 0.09" rpy=" 0 0 0"/>
       <geometry>
-        <box size=".20 .08 .15"/>
+        <!--box size=".20 .08 .15"/-->
+        <mesh filename = "package://revvyframework_ros/meshes/revvy_jetbot.dae"/>
       </geometry>
     </visual>
@@ -63,5 +64,6 @@
       <origin xyz="0.0 0 0" rpy=" 0 1.5708 1.5708"/>
       <geometry>
-        <cylinder radius = ".035" length = ".03"/>
+        <!--cylinder radius = ".035" length = ".03"/-->
+        <mesh filename = "package://revvyframework_ros/meshes/wheel.dae" scale="1.08 1.08 1.08"/>
       </geometry>
     </visual>
@@ -95,5 +97,6 @@
       <origin xyz="0.0 0 0" rpy=" 0 1.5708 1.5708"/>
       <geometry>
-        <cylinder radius = ".035" length = ".03"/>
+        <!--cylinder radius = ".035" length = ".03"/-->
+        <mesh filename = "package://revvyframework_ros/meshes/wheel.dae" scale="1.08 1.08 1.08"/>
       </geometry>
     </visual>
@@ -125,7 +128,8 @@
     </collision>
     <visual name='front_right_wheel_visual'>
-      <origin xyz="0.0 0 0" rpy=" 0 1.5708 1.5708"/>
-      <geometry>
-        <cylinder radius = ".035" length = ".03"/>
+      <origin xyz="0.0 0 0" rpy=" 0 1.5708 -1.5708"/>
+      <geometry>
+        <!--cylinder radius = ".035" length = ".03"/-->
+        <mesh filename = "package://revvyframework_ros/meshes/wheel.dae" scale="1.08 1.08 1.08"/>
       </geometry>
     </visual>
@@ -157,7 +161,8 @@
     </collision>
     <visual name='rear_right_wheel_visual'>
-      <origin xyz="0.0 0 0" rpy=" 0 1.5708 1.5708"/>
-      <geometry>
-        <cylinder radius = ".035" length = ".03"/>
+      <origin xyz="0.0 0 0" rpy=" 0 1.5708 -1.5708"/>
+      <geometry>
+        <!--cylinder radius = ".035" length = ".03"/-->
+        <mesh filename = "package://revvyframework_ros/meshes/wheel.dae" scale="1.08 1.08 1.08"/>
       </geometry>
     </visual>
@@ -189,13 +194,14 @@
       </geometry>
     </collision>
-    <visual name='camera_link_visual'>
-      <origin xyz="0 0 0" rpy=" 0 0 0"/>
-      <geometry>
-        <box size=".05 .05 .05"/>
+    <visual name='rgbd_camera_link_visual'>
+      <origin xyz="0 0 0" rpy=" 0 0 0"/>
+      <geometry>
+        <!--box size=".05 .05 .05"/-->
+        <mesh filename = "package://revvyframework_ros/meshes/d435.dae"/>
       </geometry>
     </visual>
   </link>
   <joint type="fixed" name="rgbd_camera_joint">
-    <origin xyz="0.1 0 0.15" rpy="0 0 0"/>
+    <origin xyz="0.08 0 0.15" rpy="0 0 0"/>
     <child link="rgbd_camera_link"/>
     <parent link="base_link"/>
@@ -251,10 +257,11 @@
       <origin xyz="0 0 0" rpy=" 0 0 0"/>
       <geometry>
-        <box size=".05 .05 .05"/>
-      </geometry>
-    </visual>
-  </link>
-  <joint type="fixed" name="camera_joint">
-    <origin xyz="0.1 0 0.10" rpy="-1.5707 0 -1.5707"/>
+        <!--box size=".05 .05 .05"/-->
+        <mesh filename = "package://revvyframework_ros/meshes/picam.dae" scale="0.001 0.001 0.001"/>
+      </geometry>
+    </visual>
+  </link>
+  <joint type="fixed" name="main_camera_joint">
+    <origin xyz="0.08 0 0.115" rpy="-1.5707 0 -1.5707"/>
     <child link="main_camera_link"/>
     <parent link="base_link"/>
@@ -279,12 +286,12 @@
     </collision>
     <visual name='scan_visual'>
-      <origin xyz="0 0 0" rpy=" 0 0 0"/>
-      <geometry>
-        <mesh filename = "package://revvyframework_ros/meshes/hokuyo.dae"/>
+      <origin xyz="0 0 0" rpy=" 0 0 3.1415"/>
+      <geometry>
+        <mesh filename = "package://revvyframework_ros/meshes/rplidar.dae"/>
       </geometry>
     </visual>
   </link>
   <joint type="fixed" name="scan_joint">
-    <origin xyz="-0.07 0 0.22" rpy="0 0 0"/>
+    <origin xyz="-0.066 0 0.23" rpy="0 0 0"/>
     <child link="scan"/>
     <parent link="base_link"/>

Commit message: upload local changes

File: urdf/jetson.xacro (robot description, xacro)
@@ -203,5 +203,5 @@
   </link>
   <joint type="fixed" name="rgbd_camera_joint">
-    <origin xyz="0.08 0 0.15" rpy="0 0 0"/>
+    <origin xyz="0.07 0 0.16" rpy="0 0 0"/>
     <child link="rgbd_camera_link"/>
     <parent link="base_link"/>
@@ -211,5 +211,5 @@
   </link>
   <joint type="fixed" name="rgbd_camera_depth_joint">
-    <origin xyz="0 0 0" rpy="0 0 0"/>
+    <origin xyz="0.01 0.0175 0.0125" rpy="0 0 0"/>
     <child link="rgbd_camera_depth_frame"/>
     <parent link="rgbd_camera_link"/>
@@ -225,5 +225,5 @@
   </link>
   <joint type="fixed" name="rgbd_camera_color_joint">
-    <origin xyz="0 0 0" rpy="0 0 0"/>
+    <origin xyz="0.01 0.0325 0.0125" rpy="0 0 0"/>
     <child link="rgbd_camera_color_frame"/>
     <parent link="rgbd_camera_link"/>
@@ -236,4 +236,32 @@
     <parent link="rgbd_camera_color_frame"/>
   </joint>
+  <link name="rgbd_camera_accel_frame">
+  </link>
+  <joint type="fixed" name="rgbd_camera_accel_joint">
+    <origin xyz="0 0.027 0.013" rpy="0 0 0"/>
+    <child link="rgbd_camera_accel_frame"/>
+    <parent link="rgbd_camera_link"/>
+  </joint>
+  <link name="rgbd_camera_accel_optical_frame">
+  </link>
+  <joint type="fixed" name="rgbd_camera_accel_optical_joint">
+    <origin xyz="0 0 0" rpy="-1.5707 0 -1.5707"/>
+    <child link="rgbd_camera_accel_optical_frame"/>
+    <parent link="rgbd_camera_accel_frame"/>
+  </joint>
+  <link name="rgbd_camera_gyro_frame">
+  </link>
+  <joint type="fixed" name="rgbd_camera_gyro_joint">
+    <origin xyz="0 0.027 0.013" rpy="0 0 0"/>
+    <child link="rgbd_camera_gyro_frame"/>
+    <parent link="rgbd_camera_link"/>
+  </joint>
+  <link name="rgbd_camera_gyro_optical_frame">
+  </link>
+  <joint type="fixed" name="rgbd_camera_gyro_optical_joint">
+    <origin xyz="0 0 0" rpy="-1.5707 0 -1.5707"/>
+    <child link="rgbd_camera_gyro_optical_frame"/>
+    <parent link="rgbd_camera_gyro_frame"/>
+  </joint>
   <!--camera-->
   <link name='main_camera_link'>
@@ -293,5 +321,5 @@
   </link>
   <joint type="fixed" name="scan_joint">
-    <origin xyz="-0.066 0 0.23" rpy="0 0 0"/>
+    <origin xyz="-0.08 0 0.225" rpy="0 0 0"/>
     <child link="scan"/>
     <parent link="base_link"/>
